Commit message: Lab 4 files, R2D2 controlling

File: src/my_r2d2/urdf/r2d2.xacro (robot description, xacro)
@@ -226,3 +226,10 @@
     <origin xyz="${.707*width+0.04} 0 ${.707*width}"/>
   </joint>
+  <link name="base_footprint">
+  </link>
+  <joint name="base_footprint_link" type="fixed">
+    <origin rpy="0 0 0" xyz="0 0 -0.45"/>
+    <parent link="base_link"/>
+    <child link="base_footprint"/>
+  </joint>
 </robot>
