Commit message: Lab 4 moving R2D2

File: src/my_r2d2/urdf/r2d2.urdf.xacro (robot description, xacro)
@@ -229,7 +229,7 @@
   </link>
   <joint name="base_footprint_link" type="fixed">
-    <origin rpy="0 0 0" xyz="0 0 -0.45"/>
-    <parent link="base_link"/>
-    <child link="base_footprint"/>
+    <origin rpy="0 0 0" xyz="0 0 0.45"/>
+    <parent link="base_footprint"/>
+    <child link="base_link"/>
   </joint>
 </robot>

Commit message: Lab 5 Camera work

File: src/my_r2d2/urdf/r2d2.urdf.xacro (robot description, xacro)
@@ -233,3 +233,10 @@
     <child link="base_link"/>
   </joint>
+  <link name="eye">
+  </link>
+  <joint name="eye_lens" type="continuous">
+    <origin rpy="0 0 1.57"/>
+    <parent link="lens"/>
+    <child link="eye"/>
+  </joint>
 </robot>
